Commit message: Added Schmalz gripper to Description

File: cvrb0609_description/urdf/cvrb0609.urdf.xacro (robot description, xacro)
@@ -5,4 +5,5 @@
 <!-- =================================================================================== -->
 <robot name="cvrb0609" xmlns:xacro="http://www.ros.org/wiki/xacro">
+  <xacro:include filename="$(find cvrb0609_description)/urdf/schmalz_ecbpmi.xacro"/>
   <xacro:macro name="cvrb0609" params="prefix">
     <!--
@@ -200,4 +201,11 @@
       <dynamics damping="0" friction="0"/>
     </joint>
+      <!-- Instantiate Schmalz_ecbpmi Gripper -->
+    <xacro:schmalz_ecbpmi
+      parent="${prefix}J6"
+      name="schmalz_ecbpmi"
+      prefix="">
+      <origin xyz="0 0 0" rpy="0 0 0" />
+    </xacro:schmalz_ecbpmi>
   </xacro:macro>
 </robot>

Commit message: add isaacsim controller

File: cvrb0609_description/urdf/cvrb0609.urdf.xacro (robot description, xacro)
@@ -66,4 +66,14 @@
       <dynamics damping="0" friction="0"/>
     </joint>
+    <transmission name="trans_1">
+      <type>transmission_interface/SimpleTransmission</type>
+      <joint name="${prefix}joint_1">
+      <hardwareInterface>hardware_interface/PositionJointInterface</hardwareInterface>
+      </joint>
+      <actuator name="motor_1">
+      <hardwareInterface>hardware_interface/PositionJointInterface</hardwareInterface>
+      <mechanicalReduction>1</mechanicalReduction>
+      </actuator>
+    </transmission>
     <link name="${prefix}J2">
       <visual>
@@ -93,4 +103,14 @@
       <dynamics damping="0" friction="0"/>
     </joint>
+      <transmission name="trans_2">
+        <type>transmission_interface/SimpleTransmission</type>
+        <joint name="${prefix}joint_2">
+        <hardwareInterface>hardware_interface/PositionJointInterface</hardwareInterface>
+        </joint>
+        <actuator name="motor_2">
+        <hardwareInterface>hardware_interface/PositionJointInterface</hardwareInterface>
+        <mechanicalReduction>1</mechanicalReduction>
+        </actuator>
+      </transmission>
     <link name="${prefix}J3">
       <visual>
@@ -120,4 +140,14 @@
       <dynamics damping="0" friction="0"/>
     </joint>
+    <transmission name="trans_3">
+      <type>transmission_interface/SimpleTransmission</type>
+      <joint name="${prefix}joint_3">
+      <hardwareInterface>hardware_interface/PositionJointInterface</hardwareInterface>
+      </joint>
+      <actuator name="motor_3">
+      <hardwareInterface>hardware_interface/PositionJointInterface</hardwareInterface>
+      <mechanicalReduction>1</mechanicalReduction>
+      </actuator>
+    </transmission>
     <link name="${prefix}J4">
       <visual>
@@ -147,4 +177,14 @@
       <dynamics damping="0" friction="0"/>
     </joint>
+    <transmission name="trans_4">
+      <type>transmission_interface/SimpleTransmission</type>
+      <joint name="${prefix}joint_4">
+      <hardwareInterface>hardware_interface/PositionJointInterface</hardwareInterface>
+      </joint>
+      <actuator name="motor_4">
+      <hardwareInterface>hardware_interface/PositionJointInterface</hardwareInterface>
+      <mechanicalReduction>1</mechanicalReduction>
+      </actuator>
+    </transmission>
     <link name="${prefix}J5">
       <visual>
@@ -174,4 +214,14 @@
       <dynamics damping="0" friction="0"/>
     </joint>
+      <transmission name="trans_5">
+      <type>transmission_interface/SimpleTransmission</type>
+      <joint name="${prefix}joint_5">
+      <hardwareInterface>hardware_interface/PositionJointInterface</hardwareInterface>
+      </joint>
+      <actuator name="motor_5">
+      <hardwareInterface>hardware_interface/PositionJointInterface</hardwareInterface>
+      <mechanicalReduction>1</mechanicalReduction>
+      </actuator>
+    </transmission>
     <link name="${prefix}J6">
       <visual>
@@ -201,4 +251,14 @@
       <dynamics damping="0" friction="0"/>
     </joint>
+    <transmission name="trans_6">
+      <type>transmission_interface/SimpleTransmission</type>
+      <joint name="${prefix}joint_6">
+      <hardwareInterface>hardware_interface/PositionJointInterface</hardwareInterface>
+      </joint>
+      <actuator name="motor_6">
+      <hardwareInterface>hardware_interface/PositionJointInterface</hardwareInterface>
+      <mechanicalReduction>1</mechanicalReduction>
+      </actuator>
+    </transmission>
       <!-- Instantiate Schmalz_ecbpmi Gripper -->
     <xacro:schmalz_ecbpmi
