Commit message: add base plate to description

File: techtory_cvrb0609_workcell_description/urdf/techtory_cvrb0609_workcell.urdf.xacro (robot description, xacro)
@@ -9,7 +9,8 @@
    <!-- Instantiate cobotta pro -->
   <xacro:cvrb0609 prefix="$(arg cvrb_prefix)"/>
+   <!-- base_plate link to cobotta link -->
   <joint name="$(arg prefix)joint_w" type="fixed">
-    <origin xyz="0.04 -0.3 0.93" rpy="0 0 0"/>
-    <parent link="world"/>
+    <origin xyz="0 0 0" rpy="0 0 0"/>
+    <parent link="robot_base_plate_link"/>
     <child link="$(arg cvrb_prefix)base_link"/>
   </joint>

Commit message: added topic based ros2 control

File: techtory_cvrb0609_workcell_description/urdf/techtory_cvrb0609_workcell.urdf.xacro (robot description, xacro)
@@ -5,4 +5,5 @@
   <xacro:arg name="parent" default="world" />
   <xacro:arg name="prefix" default="" />
+  <xacro:arg name="isaac_control" default="false" />
   <link name="$(arg parent)" />
   <xacro:arg name="cvrb_prefix" default="cobotta_pro_"/>
@@ -18,3 +19,66 @@
     <origin xyz="0 0 0" rpy="0 0 0" />
   </xacro:techtory_cell>
+  <xacro:if value="$(arg isaac_control)">
+    <ros2_control name="techtory_cvrb0609_workcell_ros2_control" type="system">
+      <hardware>
+        <plugin>topic_based_ros2_control/TopicBasedSystem</plugin>
+        <param name="joint_commands_topic">isaac_joint_commands</param>
+        <param name="joint_states_topic">isaac_joint_states</param>
+      </hardware>
+      <joint name="$(arg cvrb_prefix)joint1">
+          <command_interface name="position" />
+          <state_interface name="position">
+            <param name="initial_value">0.0</param>
+          </state_interface>
+          <state_interface name="velocity">
+              <param name="initial_value">0.0</param>
+          </state_interface>
+      </joint>
+      <joint name="$(arg cvrb_prefix)joint2">
+          <command_interface name="position" />
+          <state_interface name="position">
+            <param name="initial_value">0.0</param>
+          </state_interface>
+          <state_interface name="velocity">
+              <param name="initial_value">0.0</param>
+          </state_interface>
+      </joint>
+      <joint name="$(arg cvrb_prefix)joint3">
+          <command_interface name="position" />
+          <state_interface name="position">
+            <param name="initial_value">0.0</param>
+          </state_interface>
+          <state_interface name="velocity">
+              <param name="initial_value">0.0</param>
+          </state_interface>
+      </joint>
+      <joint name="$(arg cvrb_prefix)joint4">
+          <command_interface name="position" />
+          <state_interface name="position">
+            <param name="initial_value">0.0</param>
+          </state_interface>
+          <state_interface name="velocity">
+              <param name="initial_value">0.0</param>
+          </state_interface>
+      </joint>
+      <joint name="$(arg cvrb_prefix)joint5">
+          <command_interface name="position" />
+          <state_interface name="position">
+            <param name="initial_value">0.0</param>
+          </state_interface>
+          <state_interface name="velocity">
+              <param name="initial_value">0.0</param>
+          </state_interface>
+      </joint>
+      <joint name="$(arg cvrb_prefix)joint6">
+          <command_interface name="position" />
+          <state_interface name="position">
+            <param name="initial_value">0.0</param>
+          </state_interface>
+          <state_interface name="velocity">
+              <param name="initial_value">0.0</param>
+          </state_interface>
+      </joint>
+    </ros2_control>
+  </xacro:if>
 </robot>

Commit message: restructured the launch file

File: techtory_cvrb0609_workcell_description/urdf/techtory_cvrb0609_workcell.urdf.xacro (robot description, xacro)
@@ -1,16 +1,37 @@
 <?xml version="1.0" encoding="utf-8"?>
 <robot name="techtory_demo_description" xmlns:xacro="http://www.ros.org/wiki/xacro">
-  <xacro:include filename="$(find cvrb0609_description)/urdf/cvrb0609.urdf.xacro"/>
   <xacro:include filename="$(find techtory_cell_description)/urdf/techtory_cell.xaco" />
+  <xacro:arg name="model" default="cvrb0609"/>
+  <xacro:include filename="$(find denso_robot_descriptions)/robots/$(arg model)/urdf/denso_robot_macro.xacro"/>
   <xacro:arg name="parent" default="world" />
   <xacro:arg name="prefix" default="" />
   <xacro:arg name="isaac_control" default="false" />
+  <!-- parameters -->
+  <xacro:arg name="namespace" default="cobotta_pro_"/>
+  <xacro:arg name="transmission_hw_interface" default=""/>
+  <!-- ros2_control related parameters -->
+  <xacro:arg name="verbose" default="false"/>
+  <xacro:arg name="sim" default="false"/>
+  <xacro:arg name="use_mock_hardware" default="false"/>
+  <xacro:arg name="ip_address" default="192.168.0.2"/>
+  <xacro:arg name="send_format" default="288"/>
+  <xacro:arg name="recv_format" default="292"/>
+  <xacro:arg name="cvrb_prefix" default="cobotta_pro_"/>
+  <!-- arm -->
+  <xacro:denso_robot
+    model="$(arg model)"
+    namespace="$(arg namespace)"
+    transmission_hw_interface="$(arg transmission_hw_interface)"
+    sim="$(arg sim)"
+    use_mock_hardware="$(arg use_mock_hardware)"
+    ip_address="$(arg ip_address)"
+    verbose="$(arg verbose)"
+    send_format="$(arg send_format)"
+    recv_format="$(arg recv_format)"
+  />
   <link name="$(arg parent)" />
-  <xacro:arg name="cvrb_prefix" default="cobotta_pro_"/>
-   <!-- Instantiate cobotta pro -->
-  <xacro:cvrb0609 prefix="$(arg cvrb_prefix)"/>
    <!-- base_plate link to cobotta link -->
   <joint name="$(arg prefix)joint_w" type="fixed">
-    <origin xyz="0 0 0" rpy="0 0 0"/>
+    <origin xyz="0 0 0" rpy="0 0 1.5708"/>
     <parent link="robot_base_plate_link"/>
     <child link="$(arg cvrb_prefix)base_link"/>
