Commit message: feat: add switchable sim backend to ros2_control xacro
Add `sim_type` parameter to the ros2_control macro to switch between
MuJoCo (`mujoco`) and Isaac Sim topic-based (`topic`) hardware plugins.
Defaults to `topic` for backwards compatibility.

File: techtory_cobotta_moveit/config/techtory_demo_description.ros2_control.xacro (robot description, xacro)
@@ -1,13 +1,17 @@
 <?xml version="1.0"?>
 <robot xmlns:xacro="http://www.ros.org/wiki/xacro">
-    <xacro:macro name="techtory_demo_description_ros2_control" params="name initial_positions_file">
+    <xacro:macro name="techtory_demo_description_ros2_control" params="name initial_positions_file sim_type:='topic'">
         <xacro:property name="initial_positions" value="${xacro.load_yaml(initial_positions_file)['initial_positions']}"/>
         <ros2_control name="${name}" type="system">
             <hardware>
-                <!-- By default, set up controllers for simulation. This won't work on real hardware -->
-                <!-- <plugin>mock_components/GenericSystem</plugin> -->
-                <plugin>topic_based_ros2_control/TopicBasedSystem</plugin>
-                <plugin name="joint_command_topic">/isaac_joint_command</plugin>
-                <plugin name="joint_state_topic">/isaac_joint_states</plugin>
+                <xacro:if value="${sim_type == 'mujoco'}">
+                    <plugin>mujoco_ros2_control/MujocoSystemInterface</plugin>
+                    <param name="mujoco_model">$(find techtory_cobotta_moveit)/description/scene.xml</param>
+                </xacro:if>
+                <xacro:if value="${sim_type == 'topic'}">
+                    <plugin>topic_based_ros2_control/TopicBasedSystem</plugin>
+                    <param name="joint_command_topic">/isaac_joint_command</param>
+                    <param name="joint_state_topic">/isaac_joint_states</param>
+                </xacro:if>
             </hardware>
             <joint name="cobotta_pro_joint_1">

File: techtory_cobotta_moveit/config/techtory_demo_description.urdf.xacro (robot description, xacro)
@@ -2,4 +2,5 @@
 <robot xmlns:xacro="http://www.ros.org/wiki/xacro" name="techtory_demo_description">
     <xacro:arg name="initial_positions_file" default="initial_positions.yaml" />
+    <xacro:arg name="isaac_control" default="true" />
     <!-- Import techtory_demo_description urdf file -->
     <xacro:include filename="$(find techtory_cvrb0609_workcell_description)/urdf/techtory_cvrb0609_workcell.urdf.xacro" />

File: techtory_cvrb0609_workcell_description/urdf/techtory_cvrb0609_workcell.urdf.xacro (robot description, xacro)
@@ -19,15 +19,22 @@
   <xacro:arg name="cvrb_prefix" default="cobotta_pro_"/>
   <!-- arm -->
-  <xacro:denso_robot
-    model="$(arg model)"
-    namespace="$(arg namespace)"
-    transmission_hw_interface="$(arg transmission_hw_interface)"
-    sim="$(arg sim)"
-    use_mock_hardware="$(arg use_mock_hardware)"
-    ip_address="$(arg ip_address)"
-    verbose="$(arg verbose)"
-    send_format="$(arg send_format)"
-    recv_format="$(arg recv_format)"
-  />
+  <!-- When isaac_control=true, only include kinematics — hardware is provided externally (e.g. moveit FakeSystem) -->
+  <xacro:if value="$(arg isaac_control)">
+    <xacro:include filename="$(find denso_robot_descriptions)/robots/$(arg model)/urdf/denso_robot_kinematics.xacro"/>
+    <xacro:denso_robot_arm_kinematics namespace="$(arg namespace)" model="$(arg model)"/>
+  </xacro:if>
+  <xacro:unless value="$(arg isaac_control)">
+    <xacro:denso_robot
+      model="$(arg model)"
+      namespace="$(arg namespace)"
+      transmission_hw_interface="$(arg transmission_hw_interface)"
+      sim="$(arg sim)"
+      use_mock_hardware="$(arg use_mock_hardware)"
+      ip_address="$(arg ip_address)"
+      verbose="$(arg verbose)"
+      send_format="$(arg send_format)"
+      recv_format="$(arg recv_format)"
+    />
+  </xacro:unless>
   <link name="$(arg parent)" />
    <!-- base_plate link to cobotta link -->
@@ -40,66 +47,3 @@
     <origin xyz="0 0 0" rpy="0 0 0" />
   </xacro:techtory_cell>
-  <xacro:if value="$(arg isaac_control)">
-    <ros2_control name="techtory_cvrb0609_workcell_ros2_control" type="system">
-      <hardware>
-        <plugin>topic_based_ros2_control/TopicBasedSystem</plugin>
-        <param name="joint_commands_topic">isaac_joint_commands</param>
-        <param name="joint_states_topic">isaac_joint_states</param>
-      </hardware>
-      <joint name="$(arg cvrb_prefix)joint1">
-          <command_interface name="position" />
-          <state_interface name="position">
-            <param name="initial_value">0.0</param>
-          </state_interface>
-          <state_interface name="velocity">
-              <param name="initial_value">0.0</param>
-          </state_interface>
-      </joint>
-      <joint name="$(arg cvrb_prefix)joint2">
-          <command_interface name="position" />
-          <state_interface name="position">
-            <param name="initial_value">0.0</param>
-          </state_interface>
-          <state_interface name="velocity">
-              <param name="initial_value">0.0</param>
-          </state_interface>
-      </joint>
-      <joint name="$(arg cvrb_prefix)joint3">
-          <command_interface name="position" />
-          <state_interface name="position">
-            <param name="initial_value">0.0</param>
-          </state_interface>
-          <state_interface name="velocity">
-              <param name="initial_value">0.0</param>
-          </state_interface>
-      </joint>
-      <joint name="$(arg cvrb_prefix)joint4">
-          <command_interface name="position" />
-          <state_interface name="position">
-            <param name="initial_value">0.0</param>
-          </state_interface>
-          <state_interface name="velocity">
-              <param name="initial_value">0.0</param>
-          </state_interface>
-      </joint>
-      <joint name="$(arg cvrb_prefix)joint5">
-          <command_interface name="position" />
-          <state_interface name="position">
-            <param name="initial_value">0.0</param>
-          </state_interface>
-          <state_interface name="velocity">
-              <param name="initial_value">0.0</param>
-          </state_interface>
-      </joint>
-      <joint name="$(arg cvrb_prefix)joint6">
-          <command_interface name="position" />
-          <state_interface name="position">
-            <param name="initial_value">0.0</param>
-          </state_interface>
-          <state_interface name="velocity">
-              <param name="initial_value">0.0</param>
-          </state_interface>
-      </joint>
-    </ros2_control>
-  </xacro:if>
 </robot>

Commit message: Connect isaac with moveit

File: techtory_cobotta_moveit/config/techtory_demo_description.ros2_control.xacro (robot description, xacro)
@@ -11,6 +11,6 @@
                 <xacro:if value="${sim_type == 'topic'}">
                     <plugin>topic_based_ros2_control/TopicBasedSystem</plugin>
-                    <param name="joint_command_topic">/isaac_joint_command</param>
-                    <param name="joint_state_topic">/isaac_joint_states</param>
+                    <param name="joint_command_topic">/topic_based_joint_commands</param>
+                    <param name="joint_state_topic">/topic_based_joint_states</param>
                 </xacro:if>
             </hardware>

File: techtory_cobotta_workcell_description/urdf/techtory_cobotta_workcell.urdf (robot description, URDF)
Before this commit: robot techtory_demo_description, 13 links, 12 joints
Links:
- removed link schmalz_ecbpmi_base_link
- removed link schmalz_ecbpmi_body_link
- removed link tool_tip
- link cobotta_pro_J1: geometry collision mesh filename=package://denso_robot_descriptions/robots/cvrb0609/meshes/J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 scale=1 1 1; visual mesh filename=package://denso_robot_descriptions/robots/cvrb0609/meshes/J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 scale=1 1 1
- link cobotta_pro_J2: geometry collision mesh filename=package://denso_robot_descriptions/robots/cvrb0609/meshes/J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 scale=1 1 1; visual mesh filename=package://denso_robot_descriptions/robots/cvrb0609/meshes/J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 scale=1 1 1
- link cobotta_pro_J3: geometry collision mesh filename=package://denso_robot_descriptions/robots/cvrb0609/meshes/J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 scale=1 1 1; visual mesh filename=package://denso_robot_descriptions/robots/cvrb0609/meshes/J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 scale=1 1 1
- link cobotta_pro_J4: geometry collision mesh filename=package://denso_robot_descriptions/robots/cvrb0609/meshes/J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 scale=1 1 1; visual mesh filename=package://denso_robot_descriptions/robots/cvrb0609/meshes/J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 scale=1 1 1
- link cobotta_pro_J5: geometry collision mesh filename=package://denso_robot_descriptions/robots/cvrb0609/meshes/J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 scale=1 1 1; visual mesh filename=package://denso_robot_descriptions/robots/cvrb0609/meshes/J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 scale=1 1 1
- link cobotta_pro_J6: geometry collision mesh filename=package://denso_robot_descriptions/robots/cvrb0609/meshes/J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 scale=1 1 1; visual mesh filename=package://denso_robot_descriptions/robots/cvrb0609/meshes/J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 scale=1 1 1
- link cobotta_pro_base_link: geometry collision mesh filename=package://denso_robot_descriptions/robots/cvrb0609/meshes/b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 scale=1 1 1; visual mesh filename=package://denso_robot_descriptions/robots/cvrb0609/meshes/b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 scale=1 1 1
Joints:
- removed joint schmalz_ecbpmi_body_joint
- removed joint schmalz_ecbpmi_cup_joint
- removed joint schmalz_ecbpmi_tip_joint
- joint joint_w: origin xyz=0 0 0 rpy=0 0 0 -> xyz=0 0 0 rpy=0 0 1.5708

File: techtory_cobotta_workcell_description/urdf/techtory_cobotta_workcell.urdf.xacro (robot description, xacro)
@@ -16,5 +16,5 @@
        mujoco      - MuJoCo physics simulation
        topic_based - topic-based ROS2 control (e.g. for external simulators) -->
-  <xacro:arg name="hardware_type" default="mock"/>
+  <xacro:arg name="hardware_type" default="topic_based"/>
   <xacro:property name="hw_type" value="$(arg hardware_type)"/>
   <!-- ros2_control related parameters (used for real/mock modes) -->

Commit message: Add acceleration

File: techtory_cobotta_moveit/config/techtory_demo_description.ros2_control.xacro (robot description, xacro)
@@ -17,4 +17,8 @@
             <joint name="cobotta_pro_joint_1">
                 <command_interface name="position"/>
+                <command_interface name="acceleration">
+                    <param name="min">0</param>
+                    <param name="max">0.310886</param>
+                </command_interface>
                 <state_interface name="position">
                   <param name="initial_value">${initial_positions['cobotta_pro_joint_1']}</param>
@@ -24,4 +28,8 @@
             <joint name="cobotta_pro_joint_2">
                 <command_interface name="position"/>
+                <command_interface name="acceleration">
+                    <param name="min">0</param>
+                     <param name="max">0.310886</param>
+                </command_interface>
                 <state_interface name="position">
                   <param name="initial_value">${initial_positions['cobotta_pro_joint_2']}</param>
@@ -31,4 +39,8 @@
             <joint name="cobotta_pro_joint_3">
                 <command_interface name="position"/>
+                <command_interface name="acceleration">
+                    <param name="min">0</param>
+                    <param name="max">0.621773</param>
+                </command_interface>
                 <state_interface name="position">
                   <param name="initial_value">${initial_positions['cobotta_pro_joint_3']}</param>
@@ -38,4 +50,8 @@
             <joint name="cobotta_pro_joint_4">
                 <command_interface name="position"/>
+                <command_interface name="acceleration">
+                    <param name="min">0</param>
+                    <param name="max">0.049741</param>
+                </command_interface>
                 <state_interface name="position">
                   <param name="initial_value">${initial_positions['cobotta_pro_joint_4']}</param>
@@ -45,4 +61,8 @@
             <joint name="cobotta_pro_joint_5">
                 <command_interface name="position"/>
+                <command_interface name="acceleration">
+                    <param name="min">0</param>
+                    <param name="max">0.690860</param>
+                </command_interface>
                 <state_interface name="position">
                   <param name="initial_value">${initial_positions['cobotta_pro_joint_5']}</param>
@@ -52,4 +72,8 @@
             <joint name="cobotta_pro_joint_6">
                 <command_interface name="position"/>
+                <command_interface name="acceleration">
+                    <param name="min">0</param>
+                    <param name="max">0.690860</param>
+                </command_interface>
                 <state_interface name="position">
                   <param name="initial_value">${initial_positions['cobotta_pro_joint_6']}</param>

File: techtory_cobotta_workcell_description/urdf/cobotta_hardware.ros2_control.xacro (robot description, xacro)
@@ -13,4 +13,8 @@
           <param name="max">4.712389</param>
         </command_interface>
+        <command_interface name="acceleration">
+            <param name="min">0</param>
+            <param name="max">0.310886</param>
+        </command_interface>
         <state_interface name="position"/>
         <state_interface name="velocity"/>
@@ -22,4 +26,8 @@
           <param name="max">2.617994</param>
         </command_interface>
+        <command_interface name="acceleration">
+          <param name="min">0</param>
+          <param name="max">0.310886</param>
+        </command_interface>
         <state_interface name="position"/>
         <state_interface name="velocity"/>
@@ -31,4 +39,8 @@
           <param name="max">2.617994</param>
         </command_interface>
+        <command_interface name="acceleration">
+          <param name="min">0</param>
+          <param name="max">0.621773</param>
+        </command_interface>
         <state_interface name="position"/>
         <state_interface name="velocity"/>
@@ -40,4 +52,8 @@
           <param name="max">4.712389</param>
         </command_interface>
+        <command_interface name="acceleration">
+          <param name="min">0</param>
+          <param name="max">0.049741</param>
+        </command_interface>
         <state_interface name="position"/>
         <state_interface name="velocity"/>
@@ -48,4 +64,8 @@
           <param name="min">-2.617994</param>
           <param name="max">2.617994</param>
+        </command_interface>
+        <command_interface name="acceleration">
+          <param name="min">0</param>
+          <param name="max">0.690860</param>
         </command_interface>
         <state_interface name="position"/>
@@ -57,4 +77,8 @@
           <param name="min">-6.283185</param>
           <param name="max">6.283185</param>
+        </command_interface>
+        <command_interface name="acceleration">
+          <param name="min">0</param>
+          <param name="max">0.690860</param>
         </command_interface>
         <state_interface name="position"/>
@@ -72,11 +96,16 @@
         <param name="joint_states_topic">/topic_based_joint_states</param>
       </hardware>
-      <joint name="${namespace}joint_1">
-        <command_interface name="position">
-          <param name="min">-4.712389</param>
-          <param name="max">4.712389</param>
-        </command_interface>
-        <state_interface name="position"/>
-        <state_interface name="velocity"/>
+            <joint name="${namespace}joint_1">
+        <command_interface name="position">
+          <param name="min">-4.712389</param>
+          <param name="max">4.712389</param>
+        </command_interface>
+        <command_interface name="acceleration">
+            <param name="min">0</param>
+            <param name="max">0.310886</param>
+        </command_interface>
+        <state_interface name="position"/>
+        <state_interface name="velocity"/>
+        <state_interface name="effort"/>
       </joint>
       <joint name="${namespace}joint_2">
@@ -85,6 +114,11 @@
           <param name="max">2.617994</param>
         </command_interface>
-        <state_interface name="position"/>
-        <state_interface name="velocity"/>
+        <command_interface name="acceleration">
+          <param name="min">0</param>
+          <param name="max">0.310886</param>
+        </command_interface>
+        <state_interface name="position"/>
+        <state_interface name="velocity"/>
+        <state_interface name="effort"/>
       </joint>
       <joint name="${namespace}joint_3">
@@ -93,6 +127,11 @@
           <param name="max">2.617994</param>
         </command_interface>
-        <state_interface name="position"/>
-        <state_interface name="velocity"/>
+        <command_interface name="acceleration">
+          <param name="min">0</param>
+          <param name="max">0.621773</param>
+        </command_interface>
+        <state_interface name="position"/>
+        <state_interface name="velocity"/>
+        <state_interface name="effort"/>
       </joint>
       <joint name="${namespace}joint_4">
@@ -101,6 +140,11 @@
           <param name="max">4.712389</param>
         </command_interface>
-        <state_interface name="position"/>
-        <state_interface name="velocity"/>
+        <command_interface name="acceleration">
+          <param name="min">0</param>
+          <param name="max">0.049741</param>
+        </command_interface>
+        <state_interface name="position"/>
+        <state_interface name="velocity"/>
+        <state_interface name="effort"/>
       </joint>
       <joint name="${namespace}joint_5">
@@ -109,6 +153,11 @@
           <param name="max">2.617994</param>
         </command_interface>
-        <state_interface name="position"/>
-        <state_interface name="velocity"/>
+        <command_interface name="acceleration">
+          <param name="min">0</param>
+          <param name="max">0.690860</param>
+        </command_interface>
+        <state_interface name="position"/>
+        <state_interface name="velocity"/>
+        <state_interface name="effort"/>
       </joint>
       <joint name="${namespace}joint_6">
@@ -117,6 +166,11 @@
           <param name="max">6.283185</param>
         </command_interface>
-        <state_interface name="position"/>
-        <state_interface name="velocity"/>
+        <command_interface name="acceleration">
+          <param name="min">0</param>
+          <param name="max">0.690860</param>
+        </command_interface>
+        <state_interface name="position"/>
+        <state_interface name="velocity"/>
+        <state_interface name="effort"/>
       </joint>
     </ros2_control>
@@ -128,11 +182,16 @@
        <plugin>mock_components/GenericSystem</plugin>
       </hardware>
-      <joint name="${namespace}joint_1">
-        <command_interface name="position">
-          <param name="min">-4.712389</param>
-          <param name="max">4.712389</param>
-        </command_interface>
-        <state_interface name="position"/>
-        <state_interface name="velocity"/>
+           <joint name="${namespace}joint_1">
+        <command_interface name="position">
+          <param name="min">-4.712389</param>
+          <param name="max">4.712389</param>
+        </command_interface>
+        <command_interface name="acceleration">
+            <param name="min">0</param>
+            <param name="max">0.310886</param>
+        </command_interface>
+        <state_interface name="position"/>
+        <state_interface name="velocity"/>
+        <state_interface name="effort"/>
       </joint>
       <joint name="${namespace}joint_2">
@@ -141,6 +200,11 @@
           <param name="max">2.617994</param>
         </command_interface>
-        <state_interface name="position"/>
-        <state_interface name="velocity"/>
+        <command_interface name="acceleration">
+          <param name="min">0</param>
+          <param name="max">0.310886</param>
+        </command_interface>
+        <state_interface name="position"/>
+        <state_interface name="velocity"/>
+        <state_interface name="effort"/>
       </joint>
       <joint name="${namespace}joint_3">
@@ -149,6 +213,11 @@
           <param name="max">2.617994</param>
         </command_interface>
-        <state_interface name="position"/>
-        <state_interface name="velocity"/>
+        <command_interface name="acceleration">
+          <param name="min">0</param>
+          <param name="max">0.621773</param>
+        </command_interface>
+        <state_interface name="position"/>
+        <state_interface name="velocity"/>
+        <state_interface name="effort"/>
       </joint>
       <joint name="${namespace}joint_4">
@@ -157,6 +226,11 @@
           <param name="max">4.712389</param>
         </command_interface>
-        <state_interface name="position"/>
-        <state_interface name="velocity"/>
+        <command_interface name="acceleration">
+          <param name="min">0</param>
+          <param name="max">0.049741</param>
+        </command_interface>
+        <state_interface name="position"/>
+        <state_interface name="velocity"/>
+        <state_interface name="effort"/>
       </joint>
       <joint name="${namespace}joint_5">
@@ -165,6 +239,11 @@
           <param name="max">2.617994</param>
         </command_interface>
-        <state_interface name="position"/>
-        <state_interface name="velocity"/>
+        <command_interface name="acceleration">
+          <param name="min">0</param>
+          <param name="max">0.690860</param>
+        </command_interface>
+        <state_interface name="position"/>
+        <state_interface name="velocity"/>
+        <state_interface name="effort"/>
       </joint>
       <joint name="${namespace}joint_6">
@@ -173,6 +252,11 @@
           <param name="max">6.283185</param>
         </command_interface>
-        <state_interface name="position"/>
-        <state_interface name="velocity"/>
+        <command_interface name="acceleration">
+          <param name="min">0</param>
+          <param name="max">0.690860</param>
+        </command_interface>
+        <state_interface name="position"/>
+        <state_interface name="velocity"/>
+        <state_interface name="effort"/>
       </joint>
     </ros2_control>
