Commit message: Add Cumotion with Cartesian Path

File: techtory_cobotta_moveit/config/techtory_demo_description.ros2_control.xacro (robot description, xacro)
@@ -18,5 +18,5 @@
                 <command_interface name="position"/>
                 <command_interface name="acceleration">
-                    <param name="min">0</param>
+                    <param name="min">-0.310886</param>
                     <param name="max">0.310886</param>
                 </command_interface>
@@ -29,5 +29,5 @@
                 <command_interface name="position"/>
                 <command_interface name="acceleration">
-                    <param name="min">0</param>
+                    <param name="min">-0.310886</param>
                      <param name="max">0.310886</param>
                 </command_interface>
@@ -40,5 +40,5 @@
                 <command_interface name="position"/>
                 <command_interface name="acceleration">
-                    <param name="min">0</param>
+                    <param name="min">-0.621773</param>
                     <param name="max">0.621773</param>
                 </command_interface>
@@ -51,5 +51,5 @@
                 <command_interface name="position"/>
                 <command_interface name="acceleration">
-                    <param name="min">0</param>
+                    <param name="min">-0.049741</param>
                     <param name="max">0.049741</param>
                 </command_interface>
@@ -62,5 +62,5 @@
                 <command_interface name="position"/>
                 <command_interface name="acceleration">
-                    <param name="min">0</param>
+                    <param name="min">-0.690860</param>
                     <param name="max">0.690860</param>
                 </command_interface>
@@ -73,5 +73,5 @@
                 <command_interface name="position"/>
                 <command_interface name="acceleration">
-                    <param name="min">0</param>
+                    <param name="min">-0.690860</param>
                     <param name="max">0.690860</param>
                 </command_interface>

File: techtory_cobotta_moveit/config/techtory_demo_description.urdf (robot description, URDF)
Before this commit: robot techtory_demo_description, 10 links, 9 joints
Links:
- added link tool_tip0
Joints:
- added joint tool_tip0_virtual_joint: type fixed, parent cobotta_pro_J6, child tool_tip0, origin xyz=0 0 0 rpy=0 0 0

File: techtory_cobotta_workcell_description/urdf/cobotta_hardware.ros2_control.xacro (robot description, xacro)
@@ -14,5 +14,5 @@
         </command_interface>
         <command_interface name="acceleration">
-            <param name="min">0</param>
+            <param name="min">-0.310886</param>
             <param name="max">0.310886</param>
         </command_interface>
@@ -27,5 +27,5 @@
         </command_interface>
         <command_interface name="acceleration">
-          <param name="min">0</param>
+          <param name="min">-0.310886</param>
           <param name="max">0.310886</param>
         </command_interface>
@@ -40,5 +40,5 @@
         </command_interface>
         <command_interface name="acceleration">
-          <param name="min">0</param>
+          <param name="min">-0.621773</param>
           <param name="max">0.621773</param>
         </command_interface>
@@ -53,5 +53,5 @@
         </command_interface>
         <command_interface name="acceleration">
-          <param name="min">0</param>
+          <param name="min">-0.049741</param>
           <param name="max">0.049741</param>
         </command_interface>
@@ -66,5 +66,5 @@
         </command_interface>
         <command_interface name="acceleration">
-          <param name="min">0</param>
+          <param name="min">-0.690860</param>
           <param name="max">0.690860</param>
         </command_interface>
@@ -79,5 +79,5 @@
         </command_interface>
         <command_interface name="acceleration">
-          <param name="min">0</param>
+          <param name="min">-0.690860</param>
           <param name="max">0.690860</param>
         </command_interface>
@@ -102,5 +102,5 @@
         </command_interface>
         <command_interface name="acceleration">
-            <param name="min">0</param>
+            <param name="min">-0.310886</param>
             <param name="max">0.310886</param>
         </command_interface>
@@ -115,5 +115,5 @@
         </command_interface>
         <command_interface name="acceleration">
-          <param name="min">0</param>
+          <param name="min">-0.310886</param>
           <param name="max">0.310886</param>
         </command_interface>
@@ -128,5 +128,5 @@
         </command_interface>
         <command_interface name="acceleration">
-          <param name="min">0</param>
+          <param name="min">-0.621773</param>
           <param name="max">0.621773</param>
         </command_interface>
@@ -141,5 +141,5 @@
         </command_interface>
         <command_interface name="acceleration">
-          <param name="min">0</param>
+          <param name="min">-0.049741</param>
           <param name="max">0.049741</param>
         </command_interface>
@@ -154,5 +154,5 @@
         </command_interface>
         <command_interface name="acceleration">
-          <param name="min">0</param>
+          <param name="min">-0.690860</param>
           <param name="max">0.690860</param>
         </command_interface>
@@ -167,5 +167,5 @@
         </command_interface>
         <command_interface name="acceleration">
-          <param name="min">0</param>
+          <param name="min">-0.690860</param>
           <param name="max">0.690860</param>
         </command_interface>
@@ -188,5 +188,5 @@
         </command_interface>
         <command_interface name="acceleration">
-            <param name="min">0</param>
+            <param name="min">-0.310886</param>
             <param name="max">0.310886</param>
         </command_interface>
@@ -201,5 +201,5 @@
         </command_interface>
         <command_interface name="acceleration">
-          <param name="min">0</param>
+          <param name="min">-0.310886</param>
           <param name="max">0.310886</param>
         </command_interface>
@@ -214,5 +214,5 @@
         </command_interface>
         <command_interface name="acceleration">
-          <param name="min">0</param>
+          <param name="min">-0.621773</param>
           <param name="max">0.621773</param>
         </command_interface>
@@ -227,5 +227,5 @@
         </command_interface>
         <command_interface name="acceleration">
-          <param name="min">0</param>
+          <param name="min">-0.049741</param>
           <param name="max">0.049741</param>
         </command_interface>
@@ -240,5 +240,5 @@
         </command_interface>
         <command_interface name="acceleration">
-          <param name="min">0</param>
+          <param name="min">-0.690860</param>
           <param name="max">0.690860</param>
         </command_interface>
@@ -253,5 +253,5 @@
         </command_interface>
         <command_interface name="acceleration">
-          <param name="min">0</param>
+          <param name="min">-0.690860</param>
           <param name="max">0.690860</param>
         </command_interface>

File: techtory_cobotta_workcell_description/urdf/techtory_cobotta_workcell.urdf (robot description, URDF)
Before this commit: robot techtory_demo_description, 10 links, 9 joints
Links:
- added link cobotta_pro_tool0
Joints:
- added joint cobotta_pro_tool0_joint: type fixed, parent cobotta_pro_J6, child cobotta_pro_tool0, origin xyz=0 0 0 rpy=0 0 0

File: techtory_cobotta_workcell_description/urdf/techtory_cobotta_workcell.urdf.xacro (robot description, xacro)
@@ -1,5 +1,5 @@
 <?xml version="1.0" encoding="utf-8"?>
 <robot name="techtory_demo_description" xmlns:xacro="http://www.ros.org/wiki/xacro">
-  <xacro:include filename="$(find techtory_cell_description)/urdf/techtory_cell.xaco" />
+  <xacro:include filename="$(find techtory_cell_description)/urdf/techtory_cell.xacro" />
   <xacro:arg name="model" default="cvrb0609"/>
   <xacro:include filename="$(find denso_robot_descriptions)/robots/$(arg model)/urdf/denso_robot_macro.xacro"/>
@@ -74,3 +74,11 @@
     <origin xyz="0 0 0" rpy="0 0 0" />
   </xacro:techtory_cell>
+  <!-- virtual end-effector link for cobotta_proJ6 -->
+<link name="cobotta_pro_tool0" />
+<joint name="cobotta_pro_tool0_joint" type="fixed">
+  <parent link="$(arg cvrb_prefix)J6" />
+  <child link="cobotta_pro_tool0" />
+  <origin xyz="0 0 0" rpy="0 0 0" />
+</joint>
+  <!-- virtual end-effector link for cobotta_proJ6 -->
 </robot>
