Commit message: fix fake harware moveit

File: techtory_cobotta_workcell_description/urdf/cobotta_hardware.ros2_control.xacro (robot description, xacro)
@@ -122,3 +122,59 @@
     </ros2_control>
   </xacro:macro>
+  <!-- mock hardware interface for the Cobotta workcell -->
+  <xacro:macro name="cobotta_mock_ros2_control" params="namespace">
+    <ros2_control name="${namespace}TopicBasedSystem" type="system">
+      <hardware>
+       <plugin>mock_components/GenericSystem</plugin>
+      </hardware>
+      <joint name="${namespace}joint_1">
+        <command_interface name="position">
+          <param name="min">-4.712389</param>
+          <param name="max">4.712389</param>
+        </command_interface>
+        <state_interface name="position"/>
+        <state_interface name="velocity"/>
+      </joint>
+      <joint name="${namespace}joint_2">
+        <command_interface name="position">
+          <param name="min">-2.617994</param>
+          <param name="max">2.617994</param>
+        </command_interface>
+        <state_interface name="position"/>
+        <state_interface name="velocity"/>
+      </joint>
+      <joint name="${namespace}joint_3">
+        <command_interface name="position">
+          <param name="min">-2.617994</param>
+          <param name="max">2.617994</param>
+        </command_interface>
+        <state_interface name="position"/>
+        <state_interface name="velocity"/>
+      </joint>
+      <joint name="${namespace}joint_4">
+        <command_interface name="position">
+          <param name="min">-4.712389</param>
+          <param name="max">4.712389</param>
+        </command_interface>
+        <state_interface name="position"/>
+        <state_interface name="velocity"/>
+      </joint>
+      <joint name="${namespace}joint_5">
+        <command_interface name="position">
+          <param name="min">-2.617994</param>
+          <param name="max">2.617994</param>
+        </command_interface>
+        <state_interface name="position"/>
+        <state_interface name="velocity"/>
+      </joint>
+      <joint name="${namespace}joint_6">
+        <command_interface name="position">
+          <param name="min">-6.283185</param>
+          <param name="max">6.283185</param>
+        </command_interface>
+        <state_interface name="position"/>
+        <state_interface name="velocity"/>
+      </joint>
+    </ros2_control>
+  </xacro:macro>
 </robot>

File: techtory_cobotta_workcell_description/urdf/techtory_cobotta_workcell.urdf.xacro (robot description, xacro)
@@ -16,5 +16,5 @@
        mujoco      - MuJoCo physics simulation
        topic_based - topic-based ROS2 control (e.g. for external simulators) -->
-  <xacro:arg name="hardware_type" default="real"/>
+  <xacro:arg name="hardware_type" default="mock"/>
   <xacro:property name="hw_type" value="$(arg hardware_type)"/>
   <!-- ros2_control related parameters (used for real/mock modes) -->
@@ -60,4 +60,8 @@
     <xacro:cobotta_topic_based_ros2_control namespace="$(arg namespace)"/>
   </xacro:if>
+    <!-- topic_based hardware plugin -->
+  <xacro:if value="${hw_type == 'mock'}">
+    <xacro:cobotta_mock_ros2_control namespace="$(arg namespace)"/>
+  </xacro:if>
   <link name="$(arg parent)" />
   <!-- base_plate link to cobotta link -->

Commit message: add onrobot_controller

File: techtory_cobotta_workcell_description/urdf/cobotta_hardware.ros2_control.xacro (robot description, xacro)
@@ -150,4 +150,13 @@
         <state_interface name="effort"/>
       </joint>
+      <joint name="rg6_finger_joint">
+      <command_interface name="position">
+        <param name="min">-0.628319</param>
+        <param name="max">0.628319</param>
+      </command_interface>
+      <state_interface name="position"/>
+      <state_interface name="velocity"/>
+      <state_interface name="effort"/>
+    </joint>
     </ros2_control>
   </xacro:macro>

Commit message: Add mock hardware interface and update launch configurations for hybrid planning

File: techtory_cobotta_workcell_description/urdf/cobotta_hardware.ros2_control.xacro (robot description, xacro)
@@ -175,5 +175,5 @@
   <!-- mock hardware interface for the Cobotta workcell -->
   <xacro:macro name="cobotta_mock_ros2_control" params="namespace">
-    <ros2_control name="${namespace}TopicBasedSystem" type="system">
+    <ros2_control name="${namespace}MockSystem" type="system">
       <hardware>
        <plugin>mock_components/GenericSystem</plugin>
@@ -184,9 +184,7 @@
           <param name="max">4.712389</param>
         </command_interface>
-        <command_interface name="acceleration">
-            <param name="min">-0.310886</param>
-            <param name="max">0.310886</param>
-        </command_interface>
-        <state_interface name="position"/>
+        <state_interface name="position">
+          <param name="initial_value">0.0</param>
+        </state_interface>
         <state_interface name="velocity"/>
         <state_interface name="effort"/>
@@ -197,9 +195,7 @@
           <param name="max">2.617994</param>
         </command_interface>
-        <command_interface name="acceleration">
-          <param name="min">-0.310886</param>
-          <param name="max">0.310886</param>
-        </command_interface>
-        <state_interface name="position"/>
+        <state_interface name="position">
+          <param name="initial_value">0.785398</param>
+        </state_interface>
         <state_interface name="velocity"/>
         <state_interface name="effort"/>
@@ -210,9 +206,7 @@
           <param name="max">2.617994</param>
         </command_interface>
-        <command_interface name="acceleration">
-          <param name="min">-0.621773</param>
-          <param name="max">0.621773</param>
-        </command_interface>
-        <state_interface name="position"/>
+        <state_interface name="position">
+          <param name="initial_value">0.349066</param>
+        </state_interface>
         <state_interface name="velocity"/>
         <state_interface name="effort"/>
@@ -223,9 +217,7 @@
           <param name="max">4.712389</param>
         </command_interface>
-        <command_interface name="acceleration">
-          <param name="min">-0.049741</param>
-          <param name="max">0.049741</param>
-        </command_interface>
-        <state_interface name="position"/>
+        <state_interface name="position">
+          <param name="initial_value">0.349066</param>
+        </state_interface>
         <state_interface name="velocity"/>
         <state_interface name="effort"/>
@@ -236,9 +228,7 @@
           <param name="max">2.617994</param>
         </command_interface>
-        <command_interface name="acceleration">
-          <param name="min">-0.690860</param>
-          <param name="max">0.690860</param>
-        </command_interface>
-        <state_interface name="position"/>
+        <state_interface name="position">
+          <param name="initial_value">0.349066</param>
+        </state_interface>
         <state_interface name="velocity"/>
         <state_interface name="effort"/>
@@ -249,7 +239,14 @@
           <param name="max">6.283185</param>
         </command_interface>
-        <command_interface name="acceleration">
-          <param name="min">-0.690860</param>
-          <param name="max">0.690860</param>
+        <state_interface name="position">
+          <param name="initial_value">0.349066</param>
+        </state_interface>
+        <state_interface name="velocity"/>
+        <state_interface name="effort"/>
+      </joint>
+      <joint name="rg6_finger_joint">
+        <command_interface name="position">
+          <param name="min">-0.628319</param>
+          <param name="max">0.628319</param>
         </command_interface>
         <state_interface name="position"/>

File: techtory_cobotta_workcell_description/urdf/techtory_cobotta_workcell.urdf.xacro (robot description, xacro)
@@ -30,11 +30,11 @@
   <xacro:arg name="recv_format" default="292"/>
   <xacro:arg name="cvrb_prefix" default="cobotta_pro_"/>
-  <!-- arm: mujoco and topic_based load kinematics only; hardware plugin added separately -->
-  <xacro:if value="${hw_type == 'mujoco' or hw_type == 'topic_based'}">
+  <!-- arm: mujoco, topic_based, and mock load kinematics only; hardware plugin added separately -->
+  <xacro:if value="${hw_type == 'mujoco' or hw_type == 'topic_based' or hw_type == 'mock'}">
     <xacro:include filename="$(find denso_robot_descriptions)/robots/$(arg model)/urdf/denso_robot_kinematics.xacro"/>
     <xacro:denso_robot_arm_kinematics namespace="$(arg namespace)" model="$(arg model)"/>
   </xacro:if>
-  <!-- real and mock modes use the denso_robot macro -->
-  <xacro:unless value="${hw_type == 'mujoco' or hw_type == 'topic_based'}">
+  <!-- real mode uses the denso_robot macro -->
+  <xacro:unless value="${hw_type == 'mujoco' or hw_type == 'topic_based' or hw_type == 'mock'}">
     <!-- When isaac_control=true, only include kinematics — hardware is provided externally (e.g. moveit FakeSystem) -->
     <xacro:if value="$(arg isaac_control)">

Commit message: add hammer

File: techtory_cobotta_workcell_description/urdf/cobotta_hardware.ros2_control.xacro (robot description, xacro)
@@ -62,4 +62,17 @@
         <state_interface name="effort"/>
       </joint>
+      <joint name="rg6_finger_joint">
+      <command_interface name="position">
+        <param name="min">-0.628319</param>
+        <param name="max">0.628319</param>
+      </command_interface>
+      <command_interface name="acceleration">
+            <param name="min">-0.310886</param>
+            <param name="max">0.310886</param>
+      </command_interface>
+      <state_interface name="position"/>
+      <state_interface name="velocity"/>
+      <state_interface name="effort"/>
+    </joint>
     </ros2_control>
   </xacro:macro>
@@ -261,4 +274,17 @@
         <state_interface name="effort"/>
       </joint>
+      <joint name="rg6_finger_joint">
+      <command_interface name="position">
+        <param name="min">-0.628319</param>
+        <param name="max">0.628319</param>
+      </command_interface>
+      <command_interface name="acceleration">
+            <param name="min">-0.310886</param>
+            <param name="max">0.310886</param>
+      </command_interface>
+      <state_interface name="position"/>
+      <state_interface name="velocity"/>
+      <state_interface name="effort"/>
+    </joint>
     </ros2_control>
   </xacro:macro>

File: techtory_cobotta_workcell_description/urdf/techtory_cobotta_workcell.urdf.xacro (robot description, xacro)
@@ -7,4 +7,5 @@
     <!-- Gripper Xacro -->
   <xacro:include filename="$(find onrobot_rg_description)/urdf/onrobot_rg6_model_macro.xacro" />
+  <xacro:include filename="$(find techtory_cobotta_workcell_description)/urdf/shelf.xacro"/>
   <xacro:arg name="parent" default="world" />
   <xacro:arg name="prefix" default="" />
@@ -99,4 +100,7 @@
     <child link="$(arg gripper_prefix)base_link"/>
   </joint>
+  <xacro:shelf prefix="shelf_" parent="$(arg parent)">
+    <origin xyz="0.61 0.27 0.94" rpy="0 0 1.5708"/>
+  </xacro:shelf>
   <!-- virtual end-effector link for cobotta_proJ6 -->
 <link name="cobotta_pro_tool0" />

File: techtory_cobotta_workcell_description/urdf/techtory_cobotta_workcell2.urdf (robot description, URDF)
Before this commit: robot techtory_demo_description, 28 links, 27 joints
Links:
- removed link camera1_link
- removed link camera1_optical_frame
- removed link shelf_base_link
- removed link shelf_board_bottom_link
- removed link shelf_board_middle_link
- removed link shelf_board_top_link
- removed link shelf_leg_back_left_link
- removed link shelf_leg_back_right_link
- removed link shelf_leg_front_left_link
- removed link shelf_leg_front_right_link
Joints:
- removed joint camera1_joint
- removed joint camera1_optical_joint
- removed joint shelf_base_joint
- removed joint shelf_board_bottom_joint
- removed joint shelf_board_middle_joint
- removed joint shelf_board_top_joint
- removed joint shelf_leg_back_left_joint
- removed joint shelf_leg_back_right_joint
- removed joint shelf_leg_front_left_joint
- removed joint shelf_leg_front_right_joint
