Commit message: Remove obsolete MJCF and URDF files for the Techtory Cobotta workcell, including material definitions and robot descriptions, to streamline the project structure and eliminate unused assets.

File: techtory_cobotta_workcell_description/urdf/cobotta_hardware.ros2_control.xacro (robot description, xacro)
@@ -1,80 +1,4 @@
 <?xml version="1.0"?>
 <robot xmlns:xacro="http://www.ros.org/wiki/xacro">
-  <!-- MuJoCo hardware interface for the Cobotta workcell -->
-  <xacro:macro name="cobotta_mujoco_ros2_control" params="namespace">
-    <ros2_control name="${namespace}MujocoSystem" type="system">
-      <hardware>
-        <plugin>mujoco_ros2_control/MujocoSystemInterface</plugin>
-        <param name="mujoco_model">$(find techtory_cobotta_workcell_description)/urdf/mjcf/scene.xml</param>
-      </hardware>
-      <joint name="${namespace}joint_1">
-        <command_interface name="position">
-          <param name="min">-4.712389</param>
-          <param name="max">4.712389</param>
-        </command_interface>
-        <state_interface name="position"/>
-        <state_interface name="velocity"/>
-        <state_interface name="effort"/>
-      </joint>
-      <joint name="${namespace}joint_2">
-        <command_interface name="position">
-          <param name="min">-2.617994</param>
-          <param name="max">2.617994</param>
-        </command_interface>
-        <state_interface name="position"/>
-        <state_interface name="velocity"/>
-        <state_interface name="effort"/>
-      </joint>
-      <joint name="${namespace}joint_3">
-        <command_interface name="position">
-          <param name="min">-2.617994</param>
-          <param name="max">2.617994</param>
-        </command_interface>
-        <state_interface name="position"/>
-        <state_interface name="velocity"/>
-        <state_interface name="effort"/>
-      </joint>
-      <joint name="${namespace}joint_4">
-        <command_interface name="position">
-          <param name="min">-4.712389</param>
-          <param name="max">4.712389</param>
-        </command_interface>
-        <state_interface name="position"/>
-        <state_interface name="velocity"/>
-        <state_interface name="effort"/>
-      </joint>
-      <joint name="${namespace}joint_5">
-        <command_interface name="position">
-          <param name="min">-2.617994</param>
-          <param name="max">2.617994</param>
-        </command_interface>
-        <state_interface name="position"/>
-        <state_interface name="velocity"/>
-        <state_interface name="effort"/>
-      </joint>
-      <joint name="${namespace}joint_6">
-        <command_interface name="position">
-          <param name="min">-6.283185</param>
-          <param name="max">6.283185</param>
-        </command_interface>
-        <state_interface name="position"/>
-        <state_interface name="velocity"/>
-        <state_interface name="effort"/>
-      </joint>
-      <joint name="finger_joint">
-      <command_interface name="position">
-        <param name="min">-0.628319</param>
-        <param name="max">0.628319</param>
-      </command_interface>
-      <command_interface name="acceleration">
-            <param name="min">-0.310886</param>
-            <param name="max">0.310886</param>
-      </command_interface>
-      <state_interface name="position"/>
-      <state_interface name="velocity"/>
-      <state_interface name="effort"/>
-    </joint>
-    </ros2_control>
-  </xacro:macro>
   <!-- Topic-based hardware interface for the Cobotta workcell -->
   <xacro:macro name="cobotta_topic_based_ros2_control" params="namespace">
