Commit message: update cell_description

File: techtory_cobotta_workcell_description/urdf/techtory_cobotta_workcell.urdf (robot description, URDF)
Before this commit: robot techtory_demo_description, 11 links, 10 joints
Links:
- added link rg6_base_link, mass 0.7; collision mesh filename=package://onrobot_rg_description/meshes/rg6/collision/base_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; visual mesh filename=package://onrobot_rg_description/meshes/rg6/visual/base_lin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
- added link rg6_left_inner_finger, mass 0.05; collision mesh filename=package://onrobot_rg_description/meshes/rg6/collision/inner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; visual mesh filename=package://onrobot_rg_description/meshes/rg6/visual/inner_fi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
- added link rg6_left_inner_knuckle, mass 0.05; collision mesh filename=package://onrobot_rg_description/meshes/rg6/collision/inner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; visual mesh filename=package://onrobot_rg_description/meshes/rg6/visual/inner_kn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
- added link rg6_left_outer_knuckle, mass 0.05; collision mesh filename=package://onrobot_rg_description/meshes/rg6/collision/outer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; visual mesh filename=package://onrobot_rg_description/meshes/rg6/visual/outer_kn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
- added link rg6_right_inner_finger, mass 0.05; collision mesh filename=package://onrobot_rg_description/meshes/rg6/collision/inner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; visual mesh filename=package://onrobot_rg_description/meshes/rg6/visual/inner_fi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
- added link rg6_right_inner_knuckle, mass 0.05; collision mesh filename=package://onrobot_rg_description/meshes/rg6/collision/inner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; visual mesh filename=package://onrobot_rg_description/meshes/rg6/visual/inner_kn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
- added link rg6_right_outer_knuckle, mass 0.05; collision mesh filename=package://onrobot_rg_description/meshes/rg6/collision/outer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; visual mesh filename=package://onrobot_rg_description/meshes/rg6/visual/outer_kn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
- link robot_base_plate_link: geometry collision mesh filename=package://techtory_cell_description/urdf/mesh/robot_base_li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 scale=1 1 1; visual mesh filename=package://techtory_cell_description/urdf/mesh/robot_base_li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 scale=1 1 1
Joints:
- added joint joint_rg6: type fixed, parent cobotta_pro_J6, child rg6_base_link, origin xyz=0 0 0 rpy=0 0 0
- added joint rg6_finger_joint: type revolute, parent rg6_base_link, child rg6_left_outer_knuckle, origin xyz=0 -0.024112 0.136813 rpy=0 0 0, axis -1 0 0, limit lower=-0.628319 upper=0.628319 effort=1000 velocity=2.0
- added joint rg6_left_inner_finger_joint: type revolute, parent rg6_left_outer_knuckle, child rg6_left_inner_finger, origin xyz=0 -0.047334999999999995 0.064495 rpy=0 0 0, axis 1 0 0, limit lower=-0.872665 upper=0.872665 effort=1000 velocity=2.0, mimic joint=rg6_finger_joint multiplier=1 offset=0
- added joint rg6_left_inner_knuckle_joint: type revolute, parent rg6_base_link, child rg6_left_inner_knuckle, origin xyz=0 -0.01272 0.159500 rpy=0 0 0.0, axis 1 0 0, limit lower=-0.628319 upper=0.628319 effort=1000 velocity=2.0, mimic joint=rg6_finger_joint multiplier=-1 offset=0
- added joint rg6_right_inner_finger_joint: type revolute, parent rg6_right_outer_knuckle, child rg6_right_inner_finger, origin xyz=0 -0.047334999999999995 0.064495 rpy=0 0 0, axis 1 0 0, limit lower=-0.872665 upper=0.872665 effort=1000 velocity=2.0, mimic joint=rg6_finger_joint multiplier=1 offset=0
- added joint rg6_right_inner_knuckle_joint: type revolute, parent rg6_base_link, child rg6_right_inner_knuckle, origin xyz=0 0.01272 0.159500 rpy=0 0 -3.141592653589793, axis 1 0 0, limit lower=-0.628319 upper=0.628319 effort=1000 velocity=2.0, mimic joint=rg6_finger_joint multiplier=-1 offset=0
- added joint rg6_right_outer_knuckle_joint: type revolute, parent rg6_base_link, child rg6_right_outer_knuckle, origin xyz=0 0.024112 0.136813 rpy=0 0 3.141592653589793, axis 1 0 0, limit lower=-0.628319 upper=0.628319 effort=1000 velocity=2.0, mimic joint=rg6_finger_joint multiplier=-1 offset=0
- joint cobotta_pro_tool0_joint: origin xyz=0 0 0 rpy=0 0 0 -> xyz=0 0 0.25 rpy=0 0 0; parent cobotta_pro_J6 -> rg6_base_link
- joint robot_base_plate_link_joint: origin xyz=0 -0.3 0.93 rpy=0 0 0 -> xyz=-0.275 -0.24 0.94 rpy=0 0 0

Commit message: Add shelf model with dimensions and initial values for joints in URDF

File: techtory_cobotta_workcell_description/urdf/techtory_cobotta_workcell.urdf (robot description, URDF)
Before this commit: robot techtory_demo_description, 18 links, 17 joints
Links:
- added link camera1_link
- added link camera1_optical_frame
- added link shelf1_base_link, mass 1.0
- added link shelf1_board_bottom_link, mass 1.0; collision box size=1.00 0.30 0.04; visual box size=1.00 0.30 0.04
- added link shelf1_board_middle_link, mass 1.0; collision box size=1.00 0.30 0.04; visual box size=1.00 0.30 0.04
- added link shelf1_board_top_link, mass 1.0; collision box size=1.00 0.30 0.04; visual box size=1.00 0.30 0.04
- added link shelf1_leg_back_left_link, mass 1.0; collision box size=0.04 0.04 0.80; visual box size=0.04 0.04 0.80
- added link shelf1_leg_back_right_link, mass 1.0; collision box size=0.04 0.04 0.80; visual box size=0.04 0.04 0.80
- added link shelf1_leg_front_left_link, mass 1.0; collision box size=0.04 0.04 0.80; visual box size=0.04 0.04 0.80
- added link shelf1_leg_front_right_link, mass 1.0; collision box size=0.04 0.04 0.80; visual box size=0.04 0.04 0.80
- link robot_base_plate_link: geometry collision mesh filename=package://techtory_cell_description/urdf/mesh/robot_base_li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 scale=0.9 0.9 1.5; visual mesh filename=package://techtory_cell_description/urdf/mesh/robot_base_li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 scale=0.9 0.9 1.5
Joints:
- added joint camera1_joint: type fixed, parent cell_link, child camera1_link, origin xyz=-0.65 0.65 2.0 rpy=0 0.785398 -0.785398
- added joint camera1_optical_joint: type fixed, parent camera1_link, child camera1_optical_frame, origin xyz=0 0 0 rpy=-1.5708 0 -1.5708
- added joint shelf1_base_joint: type fixed, parent world, child shelf1_base_link, origin xyz=0.61 0.27 0.9 rpy=0 0 1.5708
- added joint shelf1_board_bottom_joint: type fixed, parent shelf1_base_link, child shelf1_board_bottom_link, origin xyz=0 0 0.14 rpy=0 0 0
- added joint shelf1_board_middle_joint: type fixed, parent shelf1_base_link, child shelf1_board_middle_link, origin xyz=0 0 0.34 rpy=0 0 0
- added joint shelf1_board_top_joint: type fixed, parent shelf1_base_link, child shelf1_board_top_link, origin xyz=0 0 0.78 rpy=0 0 0
- added joint shelf1_leg_back_left_joint: type fixed, parent shelf1_base_link, child shelf1_leg_back_left_link, origin xyz=-0.48 0.13 0.40 rpy=0 0 0
- added joint shelf1_leg_back_right_joint: type fixed, parent shelf1_base_link, child shelf1_leg_back_right_link, origin xyz=-0.48 -0.13 0.40 rpy=0 0 0
- added joint shelf1_leg_front_left_joint: type fixed, parent shelf1_base_link, child shelf1_leg_front_left_link, origin xyz=0.48 0.13 0.40 rpy=0 0 0
- added joint shelf1_leg_front_right_joint: type fixed, parent shelf1_base_link, child shelf1_leg_front_right_link, origin xyz=0.48 -0.13 0.40 rpy=0 0 0
- joint robot_base_plate_link_joint: origin xyz=-0.275 -0.24 0.94 rpy=0 0 0 -> xyz=0 -0.3 0.93 rpy=0 0 0

Commit message: update trajectory

File: techtory_cobotta_workcell_description/urdf/techtory_cobotta_workcell.urdf (robot description, URDF)
Before this commit: robot techtory_demo_description, 36 links, 35 joints
Links:
- removed link shelf1_base_link
- removed link shelf1_board_bottom_link
- removed link shelf1_board_middle_link
- removed link shelf1_board_top_link
- removed link shelf1_leg_back_left_link
- removed link shelf1_leg_back_right_link
- removed link shelf1_leg_front_left_link
- removed link shelf1_leg_front_right_link
- link robot_base_plate_link: geometry collision mesh filename=package://techtory_cell_description/urdf/mesh/robot_base_li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 scale=1 1 1; visual mesh filename=package://techtory_cell_description/urdf/mesh/robot_base_li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 scale=1 1 1
- link shelf_base_link: mass None -> 1.0
- link shelf_board_bottom_link: mass None -> 1.0
- link shelf_board_middle_link: mass None -> 1.0
- link shelf_board_top_link: mass None -> 1.0
- link shelf_leg_back_left_link: mass None -> 1.0
- link shelf_leg_back_right_link: mass None -> 1.0
- link shelf_leg_front_left_link: mass None -> 1.0
- link shelf_leg_front_right_link: mass None -> 1.0
Joints:
- removed joint shelf1_base_joint
- removed joint shelf1_board_bottom_joint
- removed joint shelf1_board_middle_joint
- removed joint shelf1_board_top_joint
- removed joint shelf1_leg_back_left_joint
- removed joint shelf1_leg_back_right_joint
- removed joint shelf1_leg_front_left_joint
- removed joint shelf1_leg_front_right_joint
- joint robot_base_plate_link_joint: origin xyz=0 -0.3 0.93 rpy=0 0 0 -> xyz=-0.275 -0.24 0.94 rpy=0 0 0
- joint shelf_base_joint: origin xyz=0.61 0.27 0.9 rpy=0 0 1.5708 -> xyz=0.61 0.27 0.94 rpy=0 0 1.5708

File: techtory_cobotta_workcell_description/urdf/techtory_cobotta_workcell.urdf.xacro (robot description, xacro)
@@ -111,7 +111,3 @@
     <origin xyz="0 0 0.25" rpy="0 0 0" />
   </joint>
-    <!-- virtual end-effector link for cobotta_proJ6 -->
-  <xacro:shelf prefix="shelf1_" parent="world">
-    <origin xyz="0.61 0.27 0.9" rpy="0 0 1.5708"/>
-  </xacro:shelf>
 </robot>
