Commit message: removed cell_link from the urdf

File: techtory_cobotta_workcell_description/urdf/techtory_cobotta_workcell.urdf.xacro (robot description, xacro)
@@ -64,14 +64,10 @@
     <xacro:cobotta_mock_ros2_control namespace="$(arg namespace)"/>
   </xacro:if>
-  <link name="$(arg parent)" />
-  <!-- base_plate link to cobotta link -->
-  <joint name="$(arg prefix)joint_w" type="fixed">
-    <origin xyz="0 0 0" rpy="0 0 1.5708"/>
-    <parent link="robot_base_plate_link"/>
-    <child link="$(arg cvrb_prefix)base_link"/>
-  </joint>
-  <xacro:techtory_cell parent="$(arg parent)" prefix="$(arg prefix)">
+<link name="world" />
+  <joint name="world_to_base" type="fixed">
+    <parent link="$(arg parent)" />
+    <child link="cobotta_pro_base_link" />
     <origin xyz="0 0 0" rpy="0 0 0" />
-  </xacro:techtory_cell>
+    </joint>
   <!-- virtual end-effector link for cobotta_proJ6 -->
 <link name="cobotta_pro_tool0" />

Commit message: Change robot alignment

File: techtory_cobotta_workcell_description/urdf/techtory_cobotta_workcell.urdf.xacro (robot description, xacro)
@@ -68,6 +68,6 @@
     <parent link="$(arg parent)" />
     <child link="cobotta_pro_base_link" />
-    <origin xyz="0 0 0" rpy="0 0 0" />
-    </joint>
+    <origin xyz="0 0 0" rpy="0 0 ${pi}" />
+  </joint>
   <!-- virtual end-effector link for cobotta_proJ6 -->
 <link name="cobotta_pro_tool0" />

Commit message: Rollback from adding techtory in planning scene
This reverts commit 73528be61828c6b501e9c784f004111a9ef8c16e.

File: techtory_cobotta_workcell_description/urdf/techtory_cobotta_workcell.urdf.xacro (robot description, xacro)
@@ -68,6 +68,6 @@
     <parent link="$(arg parent)" />
     <child link="cobotta_pro_base_link" />
-    <origin xyz="0 0 0" rpy="0 0 ${pi}" />
-  </joint>
+    <origin xyz="0 0 0" rpy="0 0 0" />
+    </joint>
   <!-- virtual end-effector link for cobotta_proJ6 -->
 <link name="cobotta_pro_tool0" />

Commit message: update robot alignment

File: techtory_cobotta_workcell_description/urdf/techtory_cobotta_workcell.urdf.xacro (robot description, xacro)
@@ -68,5 +68,5 @@
     <parent link="$(arg parent)" />
     <child link="cobotta_pro_base_link" />
-    <origin xyz="0 0 0" rpy="0 0 ${pi}" />
+    <origin xyz="0 0 0" rpy="0 0 ${pi/2}" />
   </joint>
   <!-- virtual end-effector link for cobotta_proJ6 -->

Commit message: update combined urdf

File: techtory_cobotta_workcell_description/urdf/techtory_cobotta_workcell.urdf.xacro (robot description, xacro)
@@ -64,5 +64,12 @@
     <xacro:cobotta_mock_ros2_control namespace="$(arg namespace)"/>
   </xacro:if>
-<link name="world" />
+  <link name="$(arg parent)" />
+  <!-- base_plate link to cobotta link -->
+  <joint name="$(arg prefix)joint_w" type="fixed">
+    <origin xyz="0 0 0" rpy="0 0 1.5708"/>
+    <parent link="robot_base_plate_link"/>
+    <child link="$(arg cvrb_prefix)base_link"/>
+  </joint>
+<<<<<<< HEAD
   <joint name="world_to_base" type="fixed">
     <parent link="$(arg parent)" />
@@ -70,4 +77,9 @@
     <origin xyz="0 0 0" rpy="0 0 ${pi/2}" />
   </joint>
+=======
+  <xacro:techtory_cell parent="$(arg parent)" prefix="$(arg prefix)">
+    <origin xyz="0 0 0" rpy="0 0 0" />
+  </xacro:techtory_cell>
+>>>>>>> parent of 639befc (removed cell_link from the urdf)
   <!-- virtual end-effector link for cobotta_proJ6 -->
 <link name="cobotta_pro_tool0" />

Commit message: remove tf transform for combined cell

File: techtory_cobotta_workcell_description/urdf/techtory_cobotta_workcell.urdf.xacro (robot description, xacro)
@@ -71,9 +71,4 @@
     <child link="$(arg cvrb_prefix)base_link"/>
   </joint>
-  <joint name="world_to_base" type="fixed">
-    <parent link="$(arg parent)" />
-    <child link="cobotta_pro_base_link" />
-    <origin xyz="0 0 0" rpy="0 0 ${pi/2}" />
-  </joint>
   <xacro:techtory_cell parent="$(arg parent)" prefix="$(arg prefix)">
     <origin xyz="0 0 0" rpy="0 0 0" />

Commit message: add rg6 gripper in workcell description

File: techtory_cobotta_workcell_description/urdf/techtory_cobotta_workcell.urdf.xacro (robot description, xacro)
@@ -5,6 +5,9 @@
   <xacro:include filename="$(find denso_robot_descriptions)/robots/$(arg model)/urdf/denso_robot_macro.xacro"/>
   <xacro:include filename="$(find techtory_cobotta_workcell_description)/urdf/cobotta_hardware.ros2_control.xacro"/>
+    <!-- Gripper Xacro -->
+  <xacro:include filename="$(find onrobot_rg_description)/urdf/onrobot_rg6_model_macro.xacro" />
   <xacro:arg name="parent" default="world" />
   <xacro:arg name="prefix" default="" />
+  <xacro:arg name="gripper_prefix" default="rg6_" />
   <xacro:arg name="isaac_control" default="false" />
   <!-- parameters -->
@@ -74,4 +77,11 @@
     <origin xyz="0 0 0" rpy="0 0 0" />
   </xacro:techtory_cell>
+  <xacro:onrobot_rg6 prefix="rg6_"/>
+  <!-- Fixed joint from cobottaJ6 to rg6_baselink -->
+  <joint name="$(arg prefix)joint_rg6" type="fixed">
+    <origin xyz="0 0 0" rpy="0 0 0"/>
+    <parent link="$(arg cvrb_prefix)J6"/>
+    <child link="$(arg gripper_prefix)base_link"/>
+  </joint>
   <!-- virtual end-effector link for cobotta_proJ6 -->
 <link name="cobotta_pro_tool0" />

Commit message: update tool0 tip loc

File: techtory_cobotta_workcell_description/urdf/techtory_cobotta_workcell.urdf.xacro (robot description, xacro)
@@ -87,7 +87,7 @@
 <link name="cobotta_pro_tool0" />
 <joint name="cobotta_pro_tool0_joint" type="fixed">
-  <parent link="$(arg cvrb_prefix)J6" />
+  <parent link="$(arg gripper_prefix)base_link" />
   <child link="cobotta_pro_tool0" />
-  <origin xyz="0 0 0" rpy="0 0 0" />
+  <origin xyz="0 0 0.25" rpy="0 0 0" />
 </joint>
   <!-- virtual end-effector link for cobotta_proJ6 -->

Commit message: Update paths and improve workcell loading for camera integration

File: techtory_cobotta_workcell_description/urdf/techtory_cobotta_workcell.urdf.xacro (robot description, xacro)
@@ -74,4 +74,11 @@
     <child link="$(arg cvrb_prefix)base_link"/>
   </joint>
+  <!-- RealSense Cameras -->
+  <joint name="camera1_joint" type="fixed">
+      <origin rpy="0 -2.35619 -2.35619" xyz="-0.65 0.65 2.0"/>
+      <parent link="cell_link"/>
+      <child link="camera1_link"/>
+  </joint>
+  <link name="camera1_link"/>
   <xacro:techtory_cell parent="$(arg parent)" prefix="$(arg prefix)">
     <origin xyz="0 0 0" rpy="0 0 0" />

Commit message: Refactor camera configuration and update URDF for optical frame integration

File: techtory_cobotta_workcell_description/urdf/techtory_cobotta_workcell.urdf.xacro (robot description, xacro)
@@ -75,10 +75,18 @@
   </joint>
   <!-- RealSense Cameras -->
+  <!-- Isaac Sim spawn: position [-0.65, 0.65, 2.0], rotation_deg [0, 45, -45] (XYZ Euler, Z-up) -->
   <joint name="camera1_joint" type="fixed">
-      <origin rpy="0 -2.35619 -2.35619" xyz="-0.65 0.65 2.0"/>
+      <origin rpy="0 0.785398 -0.785398" xyz="-0.65 0.65 2.0"/>
       <parent link="cell_link"/>
       <child link="camera1_link"/>
   </joint>
   <link name="camera1_link"/>
+  <!-- ROS optical frame: +Z forward, +X right, +Y down (rotates camera_link by -90° X, -90° Z) -->
+  <joint name="camera1_optical_joint" type="fixed">
+      <origin rpy="-1.5708 0 -1.5708" xyz="0 0 0"/>
+      <parent link="camera1_link"/>
+      <child link="camera1_optical_frame"/>
+  </joint>
+  <link name="camera1_optical_frame"/>
   <xacro:techtory_cell parent="$(arg parent)" prefix="$(arg prefix)">
     <origin xyz="0 0 0" rpy="0 0 0" />

Commit message: Refactor Cobotta Bringup and Remove Hybrid Planning Package
- Updated the robot controller from `denso_joint_trajectory_controller` to `denso_joint_group_position_controller` in the launch file.
- Added `use_sim_time` parameter to the robot state publisher.
- Commented out the move group node in the launch description.
- Deleted the `techtory_cobotta_hybrid_planning` package, including its CMakeLists.txt, README.md, launch files, source code, and package.xml.
- Removed hybrid planning configuration files from `techtory_cobotta_moveit`.
- Added a new shelf model to the workcell description.
- Updated the workcell URDF to include the new shelf model.

File: techtory_cobotta_workcell_description/urdf/techtory_cobotta_workcell.urdf.xacro (robot description, xacro)
@@ -5,4 +5,5 @@
   <xacro:include filename="$(find denso_robot_descriptions)/robots/$(arg model)/urdf/denso_robot_macro.xacro"/>
   <xacro:include filename="$(find techtory_cobotta_workcell_description)/urdf/cobotta_hardware.ros2_control.xacro"/>
+  <xacro:include filename="$(find techtory_cobotta_workcell_description)/urdf/shelf.xacro"/>
     <!-- Gripper Xacro -->
   <xacro:include filename="$(find onrobot_rg_description)/urdf/onrobot_rg6_model_macro.xacro" />
@@ -100,10 +101,13 @@
   </joint>
   <!-- virtual end-effector link for cobotta_proJ6 -->
-<link name="cobotta_pro_tool0" />
-<joint name="cobotta_pro_tool0_joint" type="fixed">
-  <parent link="$(arg gripper_prefix)base_link" />
-  <child link="cobotta_pro_tool0" />
-  <origin xyz="0 0 0.25" rpy="0 0 0" />
-</joint>
-  <!-- virtual end-effector link for cobotta_proJ6 -->
+  <link name="cobotta_pro_tool0" />
+  <joint name="cobotta_pro_tool0_joint" type="fixed">
+    <parent link="$(arg gripper_prefix)base_link" />
+    <child link="cobotta_pro_tool0" />
+    <origin xyz="0 0 0.25" rpy="0 0 0" />
+  </joint>
+    <!-- virtual end-effector link for cobotta_proJ6 -->
+  <xacro:shelf prefix="shelf1_" parent="world">
+    <origin xyz="0.61 0.27 0.9" rpy="0 0 1.5708"/>
+  </xacro:shelf>
 </robot>

Commit message: updated poses until place

File: techtory_cobotta_workcell_description/urdf/techtory_cobotta_workcell.urdf.xacro (robot description, xacro)
@@ -109,5 +109,5 @@
     <parent link="$(arg gripper_prefix)base_link" />
     <child link="cobotta_pro_tool0" />
-    <origin xyz="0 0 0.25" rpy="0 0 0" />
+    <origin xyz="0 0 0.10" rpy="0 0 0" />
   </joint>
 </robot>
