Commit message: add pallet-box

File: techtory_cobotta_workcell_description/urdf/techtory_cobotta_workcell.urdf.xacro (robot description, xacro)
@@ -9,4 +9,5 @@
   <xacro:include filename="$(find onrobot_rg_description)/urdf/onrobot_rg6_model_macro.xacro" />
   <xacro:include filename="$(find techtory_cobotta_workcell_description)/urdf/shelf.xacro"/>
+  <xacro:include filename="$(find techtory_cobotta_workcell_description)/urdf/pallet.urdf"/>
   <xacro:arg name="parent" default="world" />
   <xacro:arg name="prefix" default="" />
@@ -84,4 +85,7 @@
   </joint>
   <link name="camera1_link"/>
+  <xacro:pallet prefix="pallet_" parent="$(arg parent)">
+    <origin xyz="-0.16 0.3 0.94" rpy="0 0 0"/>
+  </xacro:pallet>
   <!-- ROS optical frame: +Z forward, +X right, +Y down (rotates camera_link by -90° X, -90° Z) -->
   <joint name="camera1_optical_joint" type="fixed">
