Commit message: Single run

File: techtory_cobotta_workcell_description/urdf/shelf.xacro (robot description, xacro)
@@ -8,6 +8,6 @@
     Board Z-centres (origin = shelf bottom):
       top    : 0.78  (top surface at z=0.80)
-      middle : 0.34  (44 cm clear space below top board bottom)
-      bottom : 0.14  (20 cm clear space below middle board bottom)
+      middle : 0.306 (top surface at z=0.326 m)
+      bottom : 0.056 (top surface at z=0.076 m)
     Usage:
       <xacro:include filename="$(find techtory_cobotta_workcell_description)/urdf/shelf.xacro"/>
@@ -86,9 +86,9 @@
     </xacro:macro>
     <!-- top board   : centre at z=0.78 (top surface flush with leg tops at z=0.80) -->
-    <!-- middle board: centre at z=0.34 (44 cm clear space below top board)         -->
-    <!-- bottom board: centre at z=0.14 (20 cm clear space below middle board)      -->
+    <!-- middle board: centre at z=0.306 (top surface at z=0.326 m) -->
+    <!-- bottom board: centre at z=0.056 (top surface at z=0.076 m) -->
     <xacro:shelf_board suffix="top"    board_z="0.78"/>
-    <xacro:shelf_board suffix="middle" board_z="0.34"/>
-    <xacro:shelf_board suffix="bottom" board_z="0.14"/>
+    <xacro:shelf_board suffix="middle" board_z="0.306"/>
+    <xacro:shelf_board suffix="bottom" board_z="0.056"/>
   </xacro:macro>
 </robot>

File: techtory_cobotta_workcell_description/urdf/techtory_cobotta_workcell.urdf (robot description, URDF)
Before this commit: robot techtory_demo_description, 28 links, 27 joints
Links:
- removed link rg6_base_link
- removed link rg6_left_inner_finger
- removed link rg6_left_inner_knuckle
- removed link rg6_left_outer_knuckle
- removed link rg6_right_inner_finger
- removed link rg6_right_inner_knuckle
- removed link rg6_right_outer_knuckle
- added link base_link, mass 0.7; collision mesh filename=package://onrobot_rg_description/meshes/rg6/collision/base_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; visual mesh filename=package://onrobot_rg_description/meshes/rg6/visual/base_lin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
- added link left_inner_finger, mass 0.05; collision mesh filename=package://onrobot_rg_description/meshes/rg6/collision/inner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; visual mesh filename=package://onrobot_rg_description/meshes/rg6/visual/inner_fi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
- added link left_inner_knuckle, mass 0.05; collision mesh filename=package://onrobot_rg_description/meshes/rg6/collision/inner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; visual mesh filename=package://onrobot_rg_description/meshes/rg6/visual/inner_kn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
- added link left_outer_knuckle, mass 0.05; collision mesh filename=package://onrobot_rg_description/meshes/rg6/collision/outer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; visual mesh filename=package://onrobot_rg_description/meshes/rg6/visual/outer_kn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
- added link right_inner_finger, mass 0.05; collision mesh filename=package://onrobot_rg_description/meshes/rg6/collision/inner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; visual mesh filename=package://onrobot_rg_description/meshes/rg6/visual/inner_fi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
- added link right_inner_knuckle, mass 0.05; collision mesh filename=package://onrobot_rg_description/meshes/rg6/collision/inner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; visual mesh filename=package://onrobot_rg_description/meshes/rg6/visual/inner_kn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
- added link right_outer_knuckle, mass 0.05; collision mesh filename=package://onrobot_rg_description/meshes/rg6/collision/outer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; visual mesh filename=package://onrobot_rg_description/meshes/rg6/visual/outer_kn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
Joints:
- removed joint rg6_finger_joint
- removed joint rg6_left_inner_finger_joint
- removed joint rg6_left_inner_knuckle_joint
- removed joint rg6_right_inner_finger_joint
- removed joint rg6_right_inner_knuckle_joint
- removed joint rg6_right_outer_knuckle_joint
- added joint finger_joint: type revolute, parent base_link, child left_outer_knuckle, origin xyz=0 -0.024112 0.136813 rpy=0 0 0, axis -1 0 0, limit lower=-0.628319 upper=0.628319 effort=1000 velocity=2.0
- added joint left_inner_finger_joint: type revolute, parent left_outer_knuckle, child left_inner_finger, origin xyz=0 -0.047334999999999995 0.064495 rpy=0 0 0, axis 1 0 0, limit lower=-0.872665 upper=0.872665 effort=1000 velocity=2.0, mimic joint=finger_joint multiplier=1 offset=0
- added joint left_inner_knuckle_joint: type revolute, parent base_link, child left_inner_knuckle, origin xyz=0 -0.01272 0.159500 rpy=0 0 0.0, axis 1 0 0, limit lower=-0.628319 upper=0.628319 effort=1000 velocity=2.0, mimic joint=finger_joint multiplier=-1 offset=0
- added joint right_inner_finger_joint: type revolute, parent right_outer_knuckle, child right_inner_finger, origin xyz=0 -0.047334999999999995 0.064495 rpy=0 0 0, axis 1 0 0, limit lower=-0.872665 upper=0.872665 effort=1000 velocity=2.0, mimic joint=finger_joint multiplier=1 offset=0
- added joint right_inner_knuckle_joint: type revolute, parent base_link, child right_inner_knuckle, origin xyz=0 0.01272 0.159500 rpy=0 0 -3.141592653589793, axis 1 0 0, limit lower=-0.628319 upper=0.628319 effort=1000 velocity=2.0, mimic joint=finger_joint multiplier=-1 offset=0
- added joint right_outer_knuckle_joint: type revolute, parent base_link, child right_outer_knuckle, origin xyz=0 0.024112 0.136813 rpy=0 0 3.141592653589793, axis 1 0 0, limit lower=-0.628319 upper=0.628319 effort=1000 velocity=2.0, mimic joint=finger_joint multiplier=-1 offset=0
- joint cobotta_pro_tool0_joint: parent rg6_base_link -> base_link
- joint joint_rg6: child rg6_base_link -> base_link
- joint joint_w: origin xyz=0 0 0 rpy=0 0 1.5708 -> xyz=0 0 0.02 rpy=0 0 1.5708

File: techtory_cobotta_workcell_description/urdf/techtory_cobotta_workcell.urdf.xacro (robot description, xacro)
@@ -11,5 +11,5 @@
   <xacro:arg name="parent" default="world" />
   <xacro:arg name="prefix" default="" />
-  <xacro:arg name="gripper_prefix" default="rg6_" />
+  <xacro:arg name="gripper_prefix" default="" />
   <xacro:arg name="isaac_control" default="false" />
   <!-- parameters -->
@@ -72,5 +72,5 @@
   <!-- base_plate link to cobotta link -->
   <joint name="$(arg prefix)joint_w" type="fixed">
-    <origin xyz="0 0 0" rpy="0 0 1.5708"/>
+    <origin xyz="0 0 0.02" rpy="0 0 1.5708"/>
     <parent link="robot_base_plate_link"/>
     <child link="$(arg cvrb_prefix)base_link"/>
@@ -94,5 +94,5 @@
     <origin xyz="0 0 0" rpy="0 0 0" />
   </xacro:techtory_cell>
-  <xacro:onrobot_rg6 prefix="rg6_"/>
+  <xacro:onrobot_rg6 prefix=""/>
   <!-- Fixed joint from cobottaJ6 to rg6_baselink -->
   <joint name="$(arg prefix)joint_rg6" type="fixed">
@@ -109,5 +109,5 @@
     <parent link="$(arg gripper_prefix)base_link" />
     <child link="cobotta_pro_tool0" />
-    <origin xyz="0 0 0.10" rpy="0 0 0" />
+    <origin xyz="0 0 0.25" rpy="0 0 0" />
   </joint>
 </robot>
