Commit message: fix robot movement and gripper usd

File: techtory_cobotta_isaacsim/assets/robots/cvrb0609_onrobot_gripper/cobotta_mit_gripper.urdf (robot description, URDF)
Before this commit: robot techtory_demo_description, 16 links, 14 joints
Links:
- removed link rg6_base_link
- removed link rg6_left_inner_finger
- removed link rg6_left_inner_knuckle
- removed link rg6_left_outer_knuckle
- removed link rg6_right_inner_finger
- removed link rg6_right_inner_knuckle
- removed link rg6_right_outer_knuckle
- added link base_link, mass 0.7; collision mesh filename=package://onrobot_rg_description/meshes/rg6/collision/base_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; visual mesh filename=package://onrobot_rg_description/meshes/rg6/visual/base_lin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
- added link left_inner_finger, mass 0.05; collision mesh filename=package://onrobot_rg_description/meshes/rg6/collision/inner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; visual mesh filename=package://onrobot_rg_description/meshes/rg6/visual/inner_fi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
- added link left_inner_knuckle, mass 0.05; collision mesh filename=package://onrobot_rg_description/meshes/rg6/collision/inner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; visual mesh filename=package://onrobot_rg_description/meshes/rg6/visual/inner_kn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
- added link left_outer_knuckle, mass 0.05; collision mesh filename=package://onrobot_rg_description/meshes/rg6/collision/outer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; visual mesh filename=package://onrobot_rg_description/meshes/rg6/visual/outer_kn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
- added link right_inner_finger, mass 0.05; collision mesh filename=package://onrobot_rg_description/meshes/rg6/collision/inner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; visual mesh filename=package://onrobot_rg_description/meshes/rg6/visual/inner_fi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
- added link right_inner_knuckle, mass 0.05; collision mesh filename=package://onrobot_rg_description/meshes/rg6/collision/inner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; visual mesh filename=package://onrobot_rg_description/meshes/rg6/visual/inner_kn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
- added link right_outer_knuckle, mass 0.05; collision mesh filename=package://onrobot_rg_description/meshes/rg6/collision/outer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; visual mesh filename=package://onrobot_rg_description/meshes/rg6/visual/outer_kn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
Joints:
- removed joint rg6_finger_joint
- removed joint rg6_left_inner_finger_joint
- removed joint rg6_left_inner_knuckle_joint
- removed joint rg6_right_inner_finger_joint
- removed joint rg6_right_inner_knuckle_joint
- removed joint rg6_right_outer_knuckle_joint
- added joint finger_joint: type revolute, parent base_link, child left_outer_knuckle, origin xyz=0 -0.024112 0.136813 rpy=0 0 0, axis -1 0 0, limit lower=-0.628319 upper=0.628319 effort=1000 velocity=2.0
- added joint left_inner_finger_joint: type revolute, parent left_outer_knuckle, child left_inner_finger, origin xyz=0 -0.047334999999999995 0.064495 rpy=0 0 0, axis 1 0 0, limit lower=-0.872665 upper=0.872665 effort=1000 velocity=2.0, mimic joint=finger_joint multiplier=1 offset=0
- added joint left_inner_knuckle_joint: type revolute, parent base_link, child left_inner_knuckle, origin xyz=0 -0.01272 0.159500 rpy=0 0 0.0, axis 1 0 0, limit lower=-0.628319 upper=0.628319 effort=1000 velocity=2.0, mimic joint=finger_joint multiplier=-1 offset=0
- added joint right_inner_finger_joint: type revolute, parent right_outer_knuckle, child right_inner_finger, origin xyz=0 -0.047334999999999995 0.064495 rpy=0 0 0, axis 1 0 0, limit lower=-0.872665 upper=0.872665 effort=1000 velocity=2.0, mimic joint=finger_joint multiplier=1 offset=0
- added joint right_inner_knuckle_joint: type revolute, parent base_link, child right_inner_knuckle, origin xyz=0 0.01272 0.159500 rpy=0 0 -3.141592653589793, axis 1 0 0, limit lower=-0.628319 upper=0.628319 effort=1000 velocity=2.0, mimic joint=finger_joint multiplier=-1 offset=0
- added joint right_outer_knuckle_joint: type revolute, parent base_link, child right_outer_knuckle, origin xyz=0 0.024112 0.136813 rpy=0 0 3.141592653589793, axis 1 0 0, limit lower=-0.628319 upper=0.628319 effort=1000 velocity=2.0, mimic joint=finger_joint multiplier=-1 offset=0
- joint cobotta_pro_tool0_joint: parent rg6_base_link -> base_link
- joint joint_rg6: child rg6_base_link -> base_link

File: techtory_cobotta_workcell_description/urdf/cobotta_hardware.ros2_control.xacro (robot description, xacro)
@@ -62,5 +62,5 @@
         <state_interface name="effort"/>
       </joint>
-      <joint name="rg6_finger_joint">
+      <joint name="finger_joint">
       <command_interface name="position">
         <param name="min">-0.628319</param>
@@ -175,5 +175,5 @@
         <state_interface name="effort"/>
       </joint>
-      <joint name="rg6_finger_joint">
+      <joint name="finger_joint">
       <command_interface name="position">
         <param name="min">-0.628319</param>
@@ -262,14 +262,5 @@
         <state_interface name="effort"/>
       </joint>
-      <joint name="rg6_finger_joint">
-        <command_interface name="position">
-          <param name="min">-0.628319</param>
-          <param name="max">0.628319</param>
-        </command_interface>
-        <state_interface name="position"/>
-        <state_interface name="velocity"/>
-        <state_interface name="effort"/>
-      </joint>
-      <joint name="rg6_finger_joint">
+      <joint name="finger_joint">
       <command_interface name="position">
         <param name="min">-0.628319</param>
